Commit message: added collisions and fixed launch of locobot arms

File: interbotix_ros_xsarms/interbotix_xsarm_descriptions/urdf/wx250s.urdf.xacro (robot description, xacro)
@@ -2,5 +2,5 @@
 <robot name="wx250s" xmlns:xacro="http://ros.org/wiki/xacro">
   <xacro:arg name="robot_name" default = "wx250s"/>
-  <xacro:arg name="base_link_frame" default="base_link"/>
+  <xacro:arg name="base_link_frame" default="base_arm_link"/>
   <xacro:arg name="show_ar_tag" default="false"/>
   <xacro:arg name="show_gripper_bar" default="true"/>
@@ -389,5 +389,5 @@
       <joint name="left_finger" type="prismatic">
         <axis xyz="0 1 0"/>
-        <limit effort="5" lower="0.015" upper="0.037" velocity="1"/>
+        <limit effort="5" lower="0.011" upper="0.042" velocity="1"/>
         <origin rpy="0 0 0" xyz="0 0 0"/>
         <parent link="$(arg robot_name)/fingers_link"/>
@@ -406,14 +406,14 @@
       <link name="$(arg robot_name)/left_finger_link">
         <visual>
-          <origin rpy="${pi} ${pi} 0" xyz="0 0.005 0"/>
+          <origin rpy="${pi} ${pi} 0" xyz="0 -0.0205 0"/>
           <geometry>
-            <mesh filename="package://interbotix_xsarm_descriptions/meshes/wx250s_meshes/wx250s_10_gripper_finger.stl" scale="0.001 0.001 0.001"/>
+            <mesh filename="package://interbotix_xsarm_descriptions/meshes/wx250s_meshes/finger_left.stl" scale="0.001 0.001 0.001"/>
           </geometry>
           <material name="interbotix_black"/>
         </visual>
         <collision>
-          <origin rpy="${pi} ${pi} 0" xyz="0 0.005 0"/>
+          <origin rpy="${pi} ${pi} 0" xyz="0 -0.205 0"/>
           <geometry>
-            <mesh filename="package://interbotix_xsarm_descriptions/meshes/wx250s_meshes/wx250s_10_gripper_finger.stl" scale="0.001 0.001 0.001"/>
+            <mesh filename="package://interbotix_xsarm_descriptions/meshes/wx250s_meshes/finger_left.stl" scale="0.001 0.001 0.001"/>
           </geometry>
         </collision>
@@ -426,5 +426,5 @@
       <joint name="right_finger" type="prismatic">
         <axis xyz="0 1 0"/>
-        <limit effort="5" lower="-0.037" upper="-0.015" velocity="1"/>
+        <limit effort="5" lower="-0.042" upper="-0.011" velocity="1"/>
         <origin rpy="0 0 0" xyz="0 0 0"/>
         <parent link="$(arg robot_name)/fingers_link"/>
@@ -446,14 +446,14 @@
       <link name="$(arg robot_name)/right_finger_link">
         <visual>
-          <origin rpy="0 ${pi} 0" xyz="0 -0.005 0"/>
+          <origin rpy="${pi} ${pi} 0" xyz="0 0.0205 0"/>
           <geometry>
-            <mesh filename="package://interbotix_xsarm_descriptions/meshes/wx250s_meshes/wx250s_10_gripper_finger.stl" scale="0.001 0.001 0.001"/>
+            <mesh filename="package://interbotix_xsarm_descriptions/meshes/wx250s_meshes/finger_right.stl" scale="0.001 0.001 0.001"/>
           </geometry>
           <material name="interbotix_black"/>
         </visual>
         <collision>
-          <origin rpy="0 ${pi} 0" xyz="0 -0.005 0"/>
+          <origin rpy="${pi} ${pi} 0" xyz="0 0.0205 0"/>
           <geometry>
-            <mesh filename="package://interbotix_xsarm_descriptions/meshes/wx250s_meshes/wx250s_10_gripper_finger.stl" scale="0.001 0.001 0.001"/>
+            <mesh filename="package://interbotix_xsarm_descriptions/meshes/wx250s_meshes/finger_right.stl" scale="0.001 0.001 0.001"/>
           </geometry>
         </collision>
@@ -466,5 +466,5 @@
       <joint name="ee_gripper" type="fixed">
         <axis xyz="1 0 0"/>
-        <origin rpy="0 0 0" xyz="0.027575 0 0"/>
+        <origin rpy="0 0 0" xyz="0.047575 0 0"/>
         <parent link="$(arg robot_name)/fingers_link"/>
         <child link="$(arg robot_name)/ee_gripper_link"/>

Commit message: the simulation has been implemented totally

File: interbotix_ros_xsarms/interbotix_xsarm_descriptions/urdf/wx250s.urdf.xacro (robot description, xacro)
@@ -9,4 +9,6 @@
   <xacro:arg name="external_urdf_loc" default=""/>
   <xacro:arg name="load_gazebo_configs" default="false"/>
+  <xacro:arg name="use_sim" default="false"/>
+  <xacro:arg name="use_actual" default="false"/>
   <xacro:property name="urdf_loc" value="$(arg external_urdf_loc)"/>
   <xacro:property name="pi_offset" value="0.00001"/>
@@ -14,5 +16,10 @@
     <xacro:include filename="$(find interbotix_xsarm_gazebo)/config/interbotix_texture.gazebo"/>
   </xacro:if>
+  <xacro:if value="$(arg use_sim)">
+  <xacro:include filename="$(find interbotix_xsarm_descriptions)/urdf/wx250s_control_sim.xacro"/>
+  </xacro:if>
+<xacro:if value="$(arg use_actual)">
   <xacro:include filename="$(find interbotix_xsarm_descriptions)/urdf/wx250s_control.xacro"/>
+  </xacro:if>
   <material name="interbotix_black">
     <texture filename="package://interbotix_xsarm_descriptions/meshes/interbotix_black.png"/>
@@ -25,4 +32,10 @@
     </joint>
   </xacro:if>
+  <link name="base_link"/>
+  <joint name="base_link_joint" type="fixed">
+    <parent link="base_link"/>
+    <origin rpy="0 0 0" xyz="0 0 0.675"/>
+    <child link="$(arg robot_name)/$(arg base_link_frame)"/>
+  </joint>
   <link name="$(arg robot_name)/$(arg base_link_frame)">
     <visual>
